File: smart-fridge-hardware/Hardware/PCB-designs/Slave-Modules/Slave_NFC.brd (EAGLE design)
At the start: 90 x 80 mm, 29 parts, among them IC1 PCF8574T, IC2 7805DT, IC3 PCF8574T, IC4 74AHC1G126DBV, J1 RJ11-2L-B, J2 RJ11-2L-B, Q1 SPB80P06P, Q2 SPB80P06P, Q3 SPB80P06P

Commit message: .brd files for SMD-desgin
Parts:
- moved IC1 0.83 mm to (59.2, 26.2)
- moved LED1 0.19 mm to (81.0, 18.4), turned to 90 degrees
Routing:
- net N$8: track 300.7 -> 225.7 mm
- net N$9: track 270.3 -> 202.0 mm
- net AGND: track 352.6 -> 311.1 mm, vias 3 -> 6
- net N$12: track 49.0 -> 58.7 mm
- net N$15: track 24.8 -> 16.4 mm
- net N$13: track 43.7 -> 50.8 mm
- net N$2: track 94.8 -> 101.7 mm, vias 2 -> 3
- net N$22: track 48.4 -> 43.4 mm
- net N$14: track 38.4 -> 42.7 mm
- net N$24: track 43.6 -> 47.6 mm
- net N$16: track 34.8 -> 38.5 mm
- net N$21: track 227.0 -> 224.4 mm
- net N$27: track 46.9 -> 44.9 mm
- net N$1: track 90.6 -> 89.3 mm, vias 0 -> 1
- net N$3: track 31.0 -> 31.8 mm
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- added copper zone on layer 1, net AGND
- added copper zone on layer 16, net AGND
