File: SmartKitchen-Emdebbed System/Hardware/PCB-designs/Master-Module/Master-Module.sch (EAGLE design)
At the start: 9 parts, among them IC2 7805DT, J1 RJ11-2L-B, J2 RJ11-2L-B, J3 RJ11-2L-B

Commit message: customizing components
Parts:
- added R3: 2k2, rcl:R-US_R0402
- added U$2: LM335, LM335:LM335
- added X1: K375M, con-power c:K375M
Connections:
- new net N$5: R3.1, U$1.A0, U$2.OUT
- net AGND: now also U$1.GND_2, U$2.GND, X1.2, X1.3
- net N$1: no longer U$1.SDA1
- net N$10: now also X1.1
- net N$21: now also R3.2
- net N$3: no longer U$1.SCL1
Other:
- note added: "5V REGULATION"
- note added: "POWER IN 12V"
- note added: "TEMPERATURE - OUT"
- note added: "ULTRASONIC SENSOR"
- note removed: "POWER"
- moved on the sheet: J3
Changed lines of the file:
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@@
 </classes>
 <parts>
-<part name="U$1" library="DUE-shield custom" deviceset="DUE(NORMAL)" device=""/>
 <part name="J3" library="con-tycoelectronics" deviceset="RJ11" device="" technology="-2L-B"/>
 <part name="J1" library="con-tycoelectronics" deviceset="RJ11" device="" technology="-2L-B"/>
@@
 <part name="R1" library="rcl" deviceset="R-US_" device="R0402" value="4k7"/>
 <part name="R2" library="rcl" deviceset="R-US_" device="R0402" value="4k7"/>
+<part name="FRAME1" library="frames" deviceset="A4L-LOC" device=""/>
+<part name="U$1" library="DUE-shield custom" deviceset="DUE(NORMAL)" device=""/>
+<part name="X1" library="con-power c" deviceset="K375M" device=""/>
+<part name="R3" library="rcl" deviceset="R-US_" device="R0402" value="2k2"/>
+<part name="U$2" library="LM335" deviceset="LM335" device=""/>
 </parts>
 <sheets>
 <sheet>
 <plain>
-<text x="220.98" y="129.54" size="1.778" layer="95" rot="R270">12V - GND - X - TX - SCL - SDA</text>
-<text x="130.81" y="200.66" size="1.778" layer="95">12V - GND - X - TX - SCL - SDA</text>
-<text x="133.35" y="205.74" size="2.54" layer="95">BUS-CONNECTION</text>
-<text x="87.63" y="200.66" size="2.54" layer="95">POWER</text>
+<text x="179.07" y="105.41" size="1.778" layer="95" rot="R270">12V - GND - X - TX - SCL - SDA</text>
+<text x="130.81" y="198.12" size="1.778" layer="95">12V - GND - X - TX - SCL - SDA</text>
+<text x="132.08" y="201.93" size="2.54" layer="95">BUS-CONNECTION</text>
+<text x="82.55" y="201.93" size="2.54" layer="95">5V REGULATION</text>
+<text x="180.34" y="146.05" size="2.54" layer="95">POWER IN 12V</text>
+<text x="185.42" y="87.63" size="2.54" layer="95">ULTRASONIC SENSOR</text>
+<text x="181.61" y="118.11" size="2.54" layer="95">TEMPERATURE - OUT</text>
 </plain>
 <instances>
-<instance part="U$1" gate="G$1" x="81.28" y="83.82"/>
-<instance part="J3" gate="G$1" x="208.28" y="114.3"/>
+<instance part="J3" gate="G$1" x="166.37" y="90.17"/>
 <instance part="J1" gate="G$1" x="133.35" y="187.96" rot="R90"/>
 <instance part="J2" gate="G$1" x="158.75" y="187.96" rot="R90"/>
@@
 <instance part="R1" gate="G$1" x="110.49" y="182.88" rot="R90"/>
 <instance part="R2" gate="G$1" x="118.11" y="182.88" rot="R90"/>
+<instance part="FRAME1" gate="G$1" x="-8.89" y="31.75"/>
+<instance part="U$1" gate="G$1" x="81.28" y="107.95"/>
+<instance part="X1" gate="G$1" x="172.72" y="139.7"/>
+<instance part="R3" gate="G$1" x="143.51" y="128.27" rot="R90"/>
+<instance part="U$2" gate="G$1" x="168.91" y="118.11"/>
 </instances>
 <busses>
@@
 <wire x1="158.75" y1="180.34" x2="153.67" y2="180.34" width="0.1524" layer="91"/>
 <junction x="153.67" y="180.34"/>
+<wire x1="158.75" y1="142.24" x2="158.75" y2="180.34" width="0.1524" layer="91"/>
+<junction x="158.75" y="180.34"/>
+<pinref part="X1" gate="G$1" pin="1"/>
+<wire x1="167.64" y1="142.24" x2="158.75" y2="142.24" width="0.1524" layer="91"/>
 </segment>
 </net>
@@
 <wire x1="166.37" y1="160.02" x2="140.97" y2="160.02" width="0.1524" layer="91"/>
 <wire x1="140.97" y1="160.02" x2="118.11" y2="160.02" width="0.1524" layer="91"/>
-<wire x1="118.11" y1="160.02" x2="59.69" y2="160.02" width="0.1524" layer="91"/>
+<wire x1="118.11" y1="160.02" x2="30.48" y2="160.02" width="0.1524" layer="91"/>
 <pinref part="J1" gate="G$1" pin="6"/>
-<wire x1="59.69" y1="160.02" x2="30.48" y2="160.02" width="0.1524" layer="91"/>
 <wire x1="140.97" y1="185.42" x2="140.97" y2="160.02" width="0.1524" layer="91"/>
 <junction x="140.97" y="160.02"/>
@@
 <wire x1="118.11" y1="177.8" x2="118.11" y2="160.02" width="0.1524" layer="91"/>
 <junction x="118.11" y="160.02"/>
-<wire x1="30.48" y1="160.02" x2="30.48" y2="78.74" width="0.1524" layer="91"/>
+<wire x1="30.48" y1="160.02" x2="30.48" y2="102.87" width="0.1524" layer="91"/>
+<wire x1="30.48" y1="102.87" x2="46.99" y2="102.87" width="0.1524" layer="91"/>
 <pinref part="U$1" gate="G$1" pin="SDA"/>
-<wire x1="30.48" y1="78.74" x2="46.99" y2="78.74" width="0.1524" layer="91"/>
-<pinref part="U$1" gate="G$1" pin="SDA1"/>
-<wire x1="59.69" y1="127" x2="59.69" y2="160.02" width="0.1524" layer="91"/>
-<junction x="59.69" y="160.02"/>
 </segment>
 </net>
@@
 <wire x1="163.83" y1="162.56" x2="138.43" y2="162.56" width="0.1524" layer="91"/>
 <wire x1="138.43" y1="162.56" x2="110.49" y2="162.56" width="0.1524" layer="91"/>
-<wire x1="110.49" y1="162.56" x2="57.15" y2="162.56" width="0.1524" layer="91"/>
+<wire x1="110.49" y1="162.56" x2="27.94" y2="162.56" width="0.1524" layer="91"/>
 <pinref part="J1" gate="G$1" pin="5"/>
-<wire x1="57.15" y1="162.56" x2="27.94" y2="162.56" width="0.1524" layer="91"/>
 <wire x1="138.43" y1="185.42" x2="138.43" y2="162.56" width="0.1524" layer="91"/>
 <junction x="138.43" y="162.56"/>
@@
 <wire x1="110.49" y1="177.8" x2="110.49" y2="162.56" width="0.1524" layer="91"/>
 <junction x="110.49" y="162.56"/>
-<wire x1="27.94" y1="162.56" x2="27.94" y2="76.2" width="0.1524" layer="91"/>
+<wire x1="27.94" y1="162.56" x2="27.94" y2="100.33" width="0.1524" layer="91"/>
+<wire x1="27.94" y1="100.33" x2="46.99" y2="100.33" width="0.1524" layer="91"/>
 <pinref part="U$1" gate="G$1" pin="SCL"/>
-<wire x1="27.94" y1="76.2" x2="46.99" y2="76.2" width="0.1524" layer="91"/>
-<pinref part="U$1" gate="G$1" pin="SCL1"/>
-<wire x1="57.15" y1="127" x2="57.15" y2="162.56" width="0.1524" layer="91"/>
-<junction x="57.15" y="162.56"/>
 </segment>
 </net>
@@
 <wire x1="118.11" y1="193.04" x2="110.49" y2="193.04" width="0.1524" layer="91"/>
 <junction x="110.49" y="193.04"/>
-<wire x1="25.4" y1="165.1" x2="25.4" y2="101.6" width="0.1524" layer="91"/>
+<wire x1="25.4" y1="165.1" x2="25.4" y2="125.73" width="0.1524" layer="91"/>
+<wire x1="25.4" y1="125.73" x2="46.99" y2="125.73" width="0.1524" layer="91"/>
 <pinref part="U$1" gate="G$1" pin="5V"/>
-<wire x1="25.4" y1="101.6" x2="46.99" y2="101.6" width="0.1524" layer="91"/>
+<junction x="105.41" y="165.1"/>
+<pinref part="R3" gate="G$1" pin="2"/>
+<wire x1="143.51" y1="165.1" x2="105.41" y2="165.1" width="0.1524" layer="91"/>
+<wire x1="143.51" y1="133.35" x2="143.51" y2="165.1" width="0.1524" layer="91"/>
 </segment>
 </net>
@@
 <wire x1="135.89" y1="185.42" x2="135.89" y2="167.64" width="0.1524" layer="91"/>
 <junction x="135.89" y="167.64"/>
-<wire x1="22.86" y1="167.64" x2="22.86" y2="55.88" width="0.1524" layer="91"/>
+<wire x1="22.86" y1="167.64" x2="22.86" y2="80.01" width="0.1524" layer="91"/>
+<wire x1="46.99" y1="80.01" x2="22.86" y2="80.01" width="0.1524" layer="91"/>
 <pinref part="U$1" gate="G$1" pin="RX0"/>
-<wire x1="46.99" y1="55.88" x2="22.86" y2="55.88" width="0.1524" layer="91"/>
 </segment>
 </net>
@@
 <pinref part="AGND4" gate="VR1" pin="AGND"/>
 <wire x1="130.81" y1="157.48" x2="130.81" y2="172.72" width="0.1524" layer="91"/>
-<wire x1="20.32" y1="172.72" x2="20.32" y2="99.06" width="0.1524" layer="91"/>
+<wire x1="20.32" y1="172.72" x2="20.32" y2="123.19" width="0.1524" layer="91"/>
+<wire x1="20.32" y1="123.19" x2="43.18" y2="123.19" width="0.1524" layer="91"/>
 <pinref part="U$1" gate="G$1" pin="GND_1"/>
-<wire x1="20.32" y1="99.06" x2="46.99" y2="99.06" width="0.1524" layer="91"/>
-</segment>
-</net>
+<wire x1="43.18" y1="123.19" x2="46.99" y2="123.19" width="0.1524" layer="91"/>
+<wire x1="156.21" y1="137.16" x2="156.21" y2="139.7" width="0.1524" layer="91"/>
+<junction x="156.21" y="172.72"/>
+<pinref part="X1" gate="G$1" pin="3"/>
+<wire x1="156.21" y1="139.7" x2="156.21" y2="172.72" width="0.1524" layer="91"/>
+<wire x1="167.64" y1="139.7" x2="156.21" y2="139.7" width="0.1524" layer="91"/>
+<junction x="156.21" y="139.7"/>
+<pinref part="X1" gate="G$1" pin="2"/>
+<wire x1="167.64" y1="137.16" x2="156.21" y2="137.16" width="0.1524" layer="91"/>
+<pinref part="U$1" gate="G$1" pin="GND_2"/>
+<wire x1="46.99" y1="120.65" x2="43.18" y2="120.65" width="0.1524" layer="91"/>
+<wire x1="43.18" y1="120.65" x2="43.18" y2="123.19" width="0.1524" layer="91"/>
+<junction x="43.18" y="123.19"/>
+<wire x1="158.75" y1="120.65" x2="156.21" y2="120.65" width="0.1524" layer="91"/>
+<wire x1="156.21" y1="120.65" x2="156.21" y2="137.16" width="0.1524" layer="91"/>
+<junction x="156.21" y="137.16"/>
+<pinref part="U$2" gate="G$1" pin="GND"/>
+</segment>
+</net>
+<net name="N$5" class="0">
+<segment>
+<wire x1="158.75" y1="118.11" x2="143.51" y2="118.11" width="0.1524" layer="91"/>
+<wire x1="143.51" y1="118.11" x2="143.51" y2="52.07" width="0.1524" layer="91"/>
+<pinref part="U$1" gate="G$1" pin="A0"/>
+<wire x1="143.51" y1="52.07" x2="64.77" y2="52.07" width="0.1524" layer="91"/>
+<wire x1="64.77" y1="52.07" x2="64.77" y2="62.23" width="0.1524" layer="91"/>
+<pinref part="R3" gate="G$1" pin="1"/>
+<wire x1="143.51" y1="118.11" x2="143.51" y2="123.19" width="0.1524" layer="91"/>
+<junction x="143.51" y="118.11"/>
+<pinref part="U$2" gate="G$1" pin="OUT"/>
+</segment>
+</net>

Commit message: PCB shield
Connections:
- new net N$6: J3.3, U$1.7
- net AGND: now also J3.4, J3.5
- net N$21: now also J3.1
Changed lines of the file:
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@@
 <instance part="R2" gate="G$1" x="118.11" y="182.88" rot="R90"/>
 <instance part="FRAME1" gate="G$1" x="-8.89" y="31.75"/>
-<instance part="U$1" gate="G$1" x="81.28" y="107.95"/>
+<instance part="U$1" gate="G$1" x="81.28" y="102.87"/>
 <instance part="X1" gate="G$1" x="172.72" y="139.7"/>
 <instance part="R3" gate="G$1" x="143.51" y="128.27" rot="R90"/>
@@
 <wire x1="118.11" y1="177.8" x2="118.11" y2="160.02" width="0.1524" layer="91"/>
 <junction x="118.11" y="160.02"/>
-<wire x1="30.48" y1="160.02" x2="30.48" y2="102.87" width="0.1524" layer="91"/>
-<wire x1="30.48" y1="102.87" x2="46.99" y2="102.87" width="0.1524" layer="91"/>
+<wire x1="30.48" y1="160.02" x2="30.48" y2="97.79" width="0.1524" layer="91"/>
+<wire x1="30.48" y1="97.79" x2="46.99" y2="97.79" width="0.1524" layer="91"/>
 <pinref part="U$1" gate="G$1" pin="SDA"/>
 </segment>
@@
 <wire x1="110.49" y1="177.8" x2="110.49" y2="162.56" width="0.1524" layer="91"/>
 <junction x="110.49" y="162.56"/>
-<wire x1="27.94" y1="162.56" x2="27.94" y2="100.33" width="0.1524" layer="91"/>
-<wire x1="27.94" y1="100.33" x2="46.99" y2="100.33" width="0.1524" layer="91"/>
+<wire x1="27.94" y1="162.56" x2="27.94" y2="95.25" width="0.1524" layer="91"/>
+<wire x1="27.94" y1="95.25" x2="46.99" y2="95.25" width="0.1524" layer="91"/>
 <pinref part="U$1" gate="G$1" pin="SCL"/>
 </segment>
@@
 <wire x1="118.11" y1="193.04" x2="110.49" y2="193.04" width="0.1524" layer="91"/>
 <junction x="110.49" y="193.04"/>
-<wire x1="25.4" y1="165.1" x2="25.4" y2="125.73" width="0.1524" layer="91"/>
-<wire x1="25.4" y1="125.73" x2="46.99" y2="125.73" width="0.1524" layer="91"/>
+<wire x1="25.4" y1="165.1" x2="25.4" y2="120.65" width="0.1524" layer="91"/>
+<wire x1="25.4" y1="120.65" x2="46.99" y2="120.65" width="0.1524" layer="91"/>
 <pinref part="U$1" gate="G$1" pin="5V"/>
 <junction x="105.41" y="165.1"/>
@@
 <wire x1="143.51" y1="165.1" x2="105.41" y2="165.1" width="0.1524" layer="91"/>
 <wire x1="143.51" y1="133.35" x2="143.51" y2="165.1" width="0.1524" layer="91"/>
+<pinref part="J3" gate="G$1" pin="1"/>
+<wire x1="163.83" y1="95.25" x2="153.67" y2="95.25" width="0.1524" layer="91"/>
+<wire x1="153.67" y1="95.25" x2="153.67" y2="165.1" width="0.1524" layer="91"/>
+<wire x1="153.67" y1="165.1" x2="143.51" y2="165.1" width="0.1524" layer="91"/>
+<junction x="143.51" y="165.1"/>
 </segment>
 </net>
@@
 <wire x1="135.89" y1="185.42" x2="135.89" y2="167.64" width="0.1524" layer="91"/>
 <junction x="135.89" y="167.64"/>
-<wire x1="22.86" y1="167.64" x2="22.86" y2="80.01" width="0.1524" layer="91"/>
-<wire x1="46.99" y1="80.01" x2="22.86" y2="80.01" width="0.1524" layer="91"/>
+<wire x1="22.86" y1="167.64" x2="22.86" y2="74.93" width="0.1524" layer="91"/>
+<wire x1="46.99" y1="74.93" x2="22.86" y2="74.93" width="0.1524" layer="91"/>
 <pinref part="U$1" gate="G$1" pin="RX0"/>
 </segment>
@@
 <pinref part="AGND4" gate="VR1" pin="AGND"/>
 <wire x1="130.81" y1="157.48" x2="130.81" y2="172.72" width="0.1524" layer="91"/>
-<wire x1="20.32" y1="172.72" x2="20.32" y2="123.19" width="0.1524" layer="91"/>
-<wire x1="20.32" y1="123.19" x2="43.18" y2="123.19" width="0.1524" layer="91"/>
+<wire x1="20.32" y1="172.72" x2="20.32" y2="118.11" width="0.1524" layer="91"/>
+<wire x1="20.32" y1="118.11" x2="43.18" y2="118.11" width="0.1524" layer="91"/>
 <pinref part="U$1" gate="G$1" pin="GND_1"/>
-<wire x1="43.18" y1="123.19" x2="46.99" y2="123.19" width="0.1524" layer="91"/>
+<wire x1="43.18" y1="118.11" x2="46.99" y2="118.11" width="0.1524" layer="91"/>
 <wire x1="156.21" y1="137.16" x2="156.21" y2="139.7" width="0.1524" layer="91"/>
 <junction x="156.21" y="172.72"/>
@@
 <wire x1="167.64" y1="137.16" x2="156.21" y2="137.16" width="0.1524" layer="91"/>
 <pinref part="U$1" gate="G$1" pin="GND_2"/>
-<wire x1="46.99" y1="120.65" x2="43.18" y2="120.65" width="0.1524" layer="91"/>
-<wire x1="43.18" y1="120.65" x2="43.18" y2="123.19" width="0.1524" layer="91"/>
-<junction x="43.18" y="123.19"/>
+<wire x1="46.99" y1="115.57" x2="43.18" y2="115.57" width="0.1524" layer="91"/>
+<wire x1="43.18" y1="115.57" x2="43.18" y2="118.11" width="0.1524" layer="91"/>
+<junction x="43.18" y="118.11"/>
 <wire x1="158.75" y1="120.65" x2="156.21" y2="120.65" width="0.1524" layer="91"/>
 <wire x1="156.21" y1="120.65" x2="156.21" y2="137.16" width="0.1524" layer="91"/>
 <junction x="156.21" y="137.16"/>
 <pinref part="U$2" gate="G$1" pin="GND"/>
+<pinref part="J3" gate="G$1" pin="4"/>
+<wire x1="163.83" y1="87.63" x2="156.21" y2="87.63" width="0.1524" layer="91"/>
+<wire x1="156.21" y1="87.63" x2="156.21" y2="120.65" width="0.1524" layer="91"/>
+<junction x="156.21" y="120.65"/>
+<pinref part="J3" gate="G$1" pin="5"/>
+<wire x1="163.83" y1="85.09" x2="156.21" y2="85.09" width="0.1524" layer="91"/>
+<wire x1="156.21" y1="85.09" x2="156.21" y2="87.63" width="0.1524" layer="91"/>
+<junction x="156.21" y="87.63"/>
 </segment>
 </net>
@@
 <segment>
 <wire x1="158.75" y1="118.11" x2="143.51" y2="118.11" width="0.1524" layer="91"/>
-<wire x1="143.51" y1="118.11" x2="143.51" y2="52.07" width="0.1524" layer="91"/>
+<wire x1="143.51" y1="118.11" x2="143.51" y2="46.99" width="0.1524" layer="91"/>
 <pinref part="U$1" gate="G$1" pin="A0"/>
-<wire x1="143.51" y1="52.07" x2="64.77" y2="52.07" width="0.1524" layer="91"/>
-<wire x1="64.77" y1="52.07" x2="64.77" y2="62.23" width="0.1524" layer="91"/>
+<wire x1="143.51" y1="46.99" x2="64.77" y2="46.99" width="0.1524" layer="91"/>
+<wire x1="64.77" y1="46.99" x2="64.77" y2="57.15" width="0.1524" layer="91"/>
 <pinref part="R3" gate="G$1" pin="1"/>
 <wire x1="143.51" y1="118.11" x2="143.51" y2="123.19" width="0.1524" layer="91"/>
@@
 </segment>
 </net>
+<net name="N$6" class="0">
+<segment>
+<pinref part="J3" gate="G$1" pin="3"/>
+<wire x1="163.83" y1="90.17" x2="151.13" y2="90.17" width="0.1524" layer="91"/>
+<wire x1="151.13" y1="90.17" x2="151.13" y2="148.59" width="0.1524" layer="91"/>
+<wire x1="151.13" y1="148.59" x2="92.71" y2="148.59" width="0.1524" layer="91"/>
+<pinref part="U$1" gate="G$1" pin="7"/>
+<wire x1="92.71" y1="148.59" x2="92.71" y2="146.05" width="0.1524" layer="91"/>
+</segment>
+</net>
