File: SmartKitchen-Emdebbed System/Hardware/PCB-designs/Master-Module/Master-Module.brd (EAGLE design)
At the start: 92.3 x 59.7 mm, 24 parts, among them IC2 7805DT, J1 RJ11-2L-B, J2 RJ11-2L-B, J3 RJ11-2L-B, J4 RJ11-2L-B, Q1 BSS123, Q2 BSS123, X1 K375M

Commit message: Adding via's
Routing:
- net AGND: track 216.5 -> 213.2 mm, vias 3 -> 18
Changed lines of the file:
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@@
 <text x="1.651" y="21.971" size="1.778" layer="1" rot="SR270">12V DC</text>
 <text x="69.9262" y="9.0932" size="1.778" layer="1" rot="SR0">I2C BUS</text>
-<text x="9.2456" y="55.2958" size="1.27" layer="1" rot="SR180">SENSOR</text>
+<text x="9.398" y="56.388" size="1.27" layer="1" rot="SR180">SENSOR</text>
 <text x="36.1442" y="32.4612" size="2.54" layer="1">DUE SHIELD</text>
 <text x="48.7426" y="8.6106" size="1.778" layer="1" rot="R90">TEMP.</text>
@@
 <wire x1="6.02" y1="24.435" x2="6.985" y2="25.4" width="1.016" layer="1"/>
 <wire x1="6.985" y1="25.4" x2="5.755" y2="25.4" width="1.016" layer="1"/>
-<wire x1="67.4116" y1="17.1704" x2="67.3862" y2="17.145" width="0.6096" layer="1"/>
 <wire x1="69.2912" y1="38.735" x2="69.2912" y2="30.7975" width="0.6096" layer="16"/>
 <wire x1="69.2912" y1="30.7975" x2="66.4337" y2="27.94" width="0.6096" layer="16"/>
@@
 <wire x1="16.51" y1="40.4876" x2="16.51" y2="42.545" width="0.6096" layer="1"/>
 <wire x1="16.51" y1="42.545" x2="15.24" y2="42.545" width="0.6096" layer="1"/>
-<wire x1="15.24" y1="42.545" x2="14.3256" y2="43.4594" width="0.6096" layer="1"/>
+<wire x1="15.24" y1="42.545" x2="13.97" y2="43.815" width="0.6096" layer="1"/>
 <wire x1="63.5508" y1="4.826" x2="61.7728" y2="3.048" width="0.6096" layer="1"/>
 <wire x1="61.7728" y1="3.048" x2="42.2148" y2="3.048" width="0.6096" layer="1"/>
@@
 <wire x1="63.5508" y1="17.145" x2="67.3862" y2="17.145" width="0.6096" layer="1"/>
 <wire x1="69.2912" y1="20.955" x2="69.2912" y2="19.05" width="0.6096" layer="1"/>
-<wire x1="69.2912" y1="19.05" x2="67.4116" y2="17.1704" width="0.6096" layer="1"/>
-<wire x1="67.4116" y1="17.1704" x2="63.3984" y2="17.1704" width="0.6096" layer="1"/>
-<wire x1="63.3984" y1="17.1704" x2="61.0108" y2="19.558" width="0.6096" layer="1"/>
-<wire x1="61.0108" y1="19.558" x2="61.0108" y2="27.9146" width="0.6096" layer="1"/>
+<wire x1="69.2912" y1="19.05" x2="67.945" y2="17.7038" width="0.6096" layer="1"/>
+<wire x1="67.4116" y1="17.1704" x2="67.945" y2="17.7038" width="0.6096" layer="1"/>
 <wire x1="61.0108" y1="27.9146" x2="61.0362" y2="27.94" width="0.6096" layer="1"/>
 <wire x1="5.89" y1="12.62" x2="9.4742" y2="12.62" width="1.27" layer="16"/>
@@
 <wire x1="9.4742" y1="2.667" x2="13.39" y2="2.667" width="1.27" layer="16"/>
 <wire x1="13.39" y1="2.667" x2="13.39" y2="2.62" width="1.27" layer="16"/>
-<polygon width="0.6096" layer="16">
-<vertex x="0.0508" y="59.6138"/>
-<vertex x="92.2274" y="59.6138"/>
-<vertex x="92.2274" y="0.0508"/>
-<vertex x="0.0508" y="0.0508"/>
-</polygon>
-<polygon width="0.6096" layer="1" isolate="0.6096">
-<vertex x="0.0508" y="59.6138"/>
-<vertex x="92.2274" y="59.6138"/>
-<vertex x="92.2274" y="0.0508"/>
-<vertex x="0.0254" y="0.0508"/>
-<vertex x="0.0254" y="59.6138"/>
-</polygon>
 <via x="69.2912" y="30.8102" extent="1-16" drill="0.6" shape="square"/>
 <contactref element="J4" pad="2"/>
@@
 <wire x1="1.69" y1="40.3742" x2="5.1308" y2="43.815" width="0.6096" layer="1"/>
 <wire x1="5.1308" y1="43.815" x2="13.97" y2="43.815" width="0.6096" layer="1"/>
-<wire x1="13.97" y1="43.815" x2="14.3256" y2="43.4594" width="0.6096" layer="1"/>
-<wire x1="69.2912" y1="30.7975" x2="69.2912" y2="30.8102" width="0" layer="19" extent="16-16"/>
+<wire x1="61.0108" y1="27.9146" x2="62.0268" y2="27.9146" width="0.6096" layer="1"/>
+<wire x1="62.0268" y1="27.9146" x2="62.7634" y2="27.178" width="0.6096" layer="1"/>
+<wire x1="62.7634" y1="27.178" x2="62.7634" y2="17.9324" width="0.6096" layer="1"/>
+<wire x1="62.7634" y1="17.9324" x2="63.5508" y2="17.145" width="0.6096" layer="1"/>
+<wire x1="67.4116" y1="17.1704" x2="67.3862" y2="17.145" width="0.6096" layer="1"/>
+<polygon width="0.3048" layer="16" isolate="0.3048">
+<vertex x="92.2274" y="59.5884"/>
+<vertex x="92.2274" y="0.0508"/>
+<vertex x="0.0508" y="0.0508"/>
+<vertex x="0.0508" y="59.5884"/>
+<vertex x="0.1016" y="59.5884"/>
+</polygon>
+<polygon width="0.3048" layer="1" isolate="0.3048">
+<vertex x="0.0508" y="59.6138"/>
+<vertex x="92.2274" y="59.6138"/>
+<vertex x="92.2274" y="0.0508"/>
+<vertex x="0.0508" y="0.0508"/>
+</polygon>
+<via x="25.781" y="50.8762" extent="1-16" drill="0.6" shape="square"/>
+<via x="43.8404" y="49.3776" extent="1-16" drill="0.6" shape="square"/>
+<via x="28.448" y="39.3192" extent="1-16" drill="0.6" shape="square"/>
+<via x="17.8054" y="33.1216" extent="1-16" drill="0.6" shape="square"/>
+<via x="88.0872" y="6.8072" extent="1-16" drill="0.6" shape="square"/>
+<via x="60.9854" y="19.4818" extent="1-16" drill="0.6" shape="square"/>
+<via x="75.6412" y="22.9616" extent="1-16" drill="0.6" shape="square"/>
+<via x="75.5396" y="40.64" extent="1-16" drill="0.6" shape="square"/>
+<via x="11.4808" y="7.6454" extent="1-16" drill="0.6" shape="square"/>
+<via x="83.6422" y="57.1754" extent="1-16" drill="0.6" shape="square"/>
+<via x="38.2524" y="42.8244" extent="1-16" drill="0.6" shape="square"/>
+<via x="20.066" y="20.2692" extent="1-16" drill="0.6" shape="square"/>
+<via x="2.8702" y="29.7688" extent="1-16" drill="0.6" shape="square"/>
+<via x="62.5602" y="35.0774" extent="1-16" drill="0.6" shape="square"/>
+<via x="28.448" y="29.0576" extent="1-16" drill="0.6" shape="square"/>
 </signal>
 <signal name="N$5">
